File: usb-uart.sch (KiCad schematic (older format))
At the start: 21 parts, among them CN1 USB4110-GF-A, CN2 30310-5002HB, SW1 CUS-12B, U1 PRTR5V0U2X, U2 FT231XQ

Commit message: Update
* USB Type Cのプルアップ抵抗のフットプリントを変更する
* USB Type Cをより基板から飛び出す
* R4を未実装にする
Parts:
- removed RN1: 5.1k, Resistor_SMD:R_Array_Convex_2x0402, symbol Device:R_Pack02
- added R1, R2: 5.1k, Resistor_SMD:R_0402_1005Metric, symbol Device:R
- R4: renamed from R2; value 0 -> DNP
- renumbered R1 to R3, R3 to R5, RN2 to RN1, RN3 to RN2
Connections:
- net GND: now also R1.1, R2.1
- net at CN1.B5 (CC2): now also R1.2
- net at CN1.A5 (CC1): now also R2.2
Changed lines of the file:
@@
 Sheet 1 1
 Title "USB UART"
-Date "2019-12-08"
-Rev "1"
+Date "2019-12-30"
+Rev "2"
 Comp ""
 Comment1 ""
@@
 L power:GND #PWR03
 U 1 1 5E0ACE24
-P 2400 4500
-F 0 "#PWR03" H 2400 4250 50  0001 C CNN
-F 1 "GND" H 2405 4327 50  0000 C CNN
-F 2 "" H 2400 4500 50  0001 C CNN
-F 3 "" H 2400 4500 50  0001 C CNN
-	1    2400 4500
-	1    0    0    -1
-$EndComp
-Wire Wire Line
-	2400 4300 2400 4400
-Wire Wire Line
-	2500 4300 2500 4400
+P 2400 4400
+F 0 "#PWR03" H 2400 4150 50  0001 C CNN
+F 1 "GND" H 2405 4227 50  0000 C CNN
+F 2 "" H 2400 4400 50  0001 C CNN
+F 3 "" H 2400 4400 50  0001 C CNN
+	1    2400 4400
+	1    0    0    -1
+$EndComp
+Wire Wire Line
+	2400 4200 2400 4300
+Wire Wire Line
+	2500 4200 2500 4300
 Wire Wire Line
 	2400 3400 2400 3900
@@
 	9400 6100 9400 6000
 $Comp
-L Device:R_Pack02 RN3
+L Device:R_Pack02 RN2
 U 1 1 5E208CB8
 P 7900 3400
-F 0 "RN3" H 7720 3446 50  0000 R CNN
+F 0 "RN2" H 7720 3446 50  0000 R CNN
 F 1 "1k" H 7720 3355 50  0000 R CNN
 F 2 "Resistor_SMD:R_Array_Convex_2x0402" V 8075 3400 50  0001 C CNN
@@
 TXLED
 $Comp
-L Device:R_Pack02 RN2
+L Device:R_Pack02 RN1
 U 1 1 5D59E14D
 P 4900 3700
-F 0 "RN2" V 5125 3700 50  0000 C CNN
+F 0 "RN1" V 5125 3700 50  0000 C CNN
 F 1 "27" V 5034 3700 50  0000 C CNN
 F 2 "Resistor_SMD:R_Array_Convex_2x0402" V 5075 3700 50  0001 C CNN
@@
 	9400 3100 9400 3200
 $Comp
-L Device:R R3
+L Device:R R5
 U 1 1 5DF24C4A
 P 9750 3200
-F 0 "R3" V 9635 3200 50  0000 C CNN
+F 0 "R5" V 9635 3200 50  0000 C CNN
 F 1 "DNP" V 9544 3200 50  0000 C CNN
 F 2 "Resistor_SMD:R_0402_1005Metric" V 9680 3200 50  0001 C CNN
@@
 	9900 3100 10200 3100
 $Comp
-L Device:R R2
+L Device:R R4
 U 1 1 5DF201BE
 P 9750 3100
-F 0 "R2" V 9957 3100 50  0000 C CNN
-F 1 "0" V 9866 3100 50  0000 C CNN
+F 0 "R4" V 9957 3100 50  0000 C CNN
+F 1 "DNP" V 9866 3100 50  0000 C CNN
 F 2 "Resistor_SMD:R_0402_1005Metric" V 9680 3100 50  0001 C CNN
 F 3 "~" H 9750 3100 50  0001 C CNN
@@
 	1    0    0    -1
 $EndComp
-$Comp
-L Device:R_Pack02 RN1
-U 1 1 5DF570C0
-P 2400 4100
-F 0 "RN1" H 2220 4146 50  0000 R CNN
-F 1 "5.1k" H 2220 4055 50  0000 R CNN
-F 2 "Resistor_SMD:R_Array_Convex_2x0402" V 2575 4100 50  0001 C CNN
-F 3 "~" H 2400 4100 50  0001 C CNN
-	1    2400 4100
-	-1   0    0    -1
-$EndComp
-Wire Wire Line
-	2500 4400 2400 4400
-Connection ~ 2400 4400
-Wire Wire Line
-	2400 4400 2400 4500
+Wire Wire Line
+	2500 4300 2400 4300
+Connection ~ 2400 4300
+Wire Wire Line
+	2400 4300 2400 4400
 Wire Wire Line
 	10000 3900 10200 3900
@@
 $EndComp
 $Comp
-L Device:R R1
+L Device:R R3
 U 1 1 5DF65C1D
 P 9150 2600
-F 0 "R1" V 9357 2600 50  0000 C CNN
+F 0 "R3" V 9357 2600 50  0000 C CNN
 F 1 "0" V 9266 2600 50  0000 C CNN
 F 2 "Resistor_SMD:R_0402_1005Metric" V 9080 2600 50  0001 C CNN
@@
 Text Notes 9650 4400 0    50   ~ 0
 UART
+$Comp
+L Device:R R1
+U 1 1 5E039A1F
+P 2400 4050
+F 0 "R1" H 2470 4004 50  0000 L CNN
+F 1 "5.1k" H 2470 4095 50  0000 L CNN
+F 2 "Resistor_SMD:R_0402_1005Metric" V 2330 4050 50  0001 C CNN
+F 3 "~" H 2400 4050 50  0001 C CNN
+	1    2400 4050
+	-1   0    0    1
+$EndComp
+$Comp
+L Device:R R2
+U 1 1 5E0442DB
+P 2500 4050
+F 0 "R2" H 2430 4004 50  0000 R CNN
+F 1 "5.1k" H 2430 4095 50  0000 R CNN
+F 2 "Resistor_SMD:R_0402_1005Metric" V 2430 4050 50  0001 C CNN
+F 3 "~" H 2500 4050 50  0001 C CNN
+	1    2500 4050
+	-1   0    0    1
+$EndComp
 $EndSCHEMATC
